File: Digital_Output_Module/kicad/Digital_Output_Module.kicad_sch (KiCad schematic)
At the start: 0 parts

Commit message: Progress on fet output channel
Parts:
- added J?: GX16-3, symbol Connector_Generic:Conn_01x03
Other:
- sheet Output Channel: file hierarchical_sheets/fet_output_channel.kicad_sch -> hierarchical_sheets/fet_output_stage.kicad_sch
Changed lines of the file:
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@@
     (comment 1 "Seth Sievers")
+  )
+  (symbol (lib_id "power:Earth") (at 144.78 55.88 0) (unit 1)
+    (in_bom yes) (on_board yes) (fields_autoplaced)
+    (property "Reference" "#PWR?" (id 0) (at 144.78 62.23 0)
+      (effects (font (size 1.27 1.27)) hide)
+    )
+    (property "Value" "Earth" (id 1) (at 144.78 59.69 0))
+    (property "Footprint" "" (id 2) (at 144.78 55.88 0)
+      (effects (font (size 1.27 1.27)) hide)
+    )
+    (property "Datasheet" "~" (id 3) (at 144.78 55.88 0)
+      (effects (font (size 1.27 1.27)) hide)
+    )
+    (pin "1")
+  )
+  (symbol (lib_id "Connector_Generic:Conn_01x03") (at 143.51 41.91 0) (unit 1)
+    (in_bom yes) (on_board yes) (fields_autoplaced)
+    (property "Reference" "J?" (id 0) (at 146.05 40.6399 0)
+      (effects (font (size 1.27 1.27)) (justify left))
+    )
+    (property "Value" "GX16-3" (id 1) (at 146.05 43.1799 0)
+      (effects (font (size 1.27 1.27)) (justify left))
+    )
+    (property "Footprint" "" (id 2) (at 143.51 41.91 0)
+      (effects (font (size 1.27 1.27)) hide)
+    )
+    (property "Datasheet" "~" (id 3) (at 143.51 41.91 0)
+      (effects (font (size 1.27 1.27)) hide)
+    )
+    (property "Seller" "https://www.amazon.com/DIYhz-Circular-Aviation-Connector-Waterproof/dp/B089YVDYDY/ref=sr_1_2_sspa?dchild=1&keywords=3%2Bpin%2Bpanel%2Bmount%2Baviation%2Bconnector&qid=1629499361&sr=8-2-spons&spLa=ZW5jcnlwdGVkUXVhbGlmaWVyPUEzN0oxVFdTTzdPUUxFJmVuY3J5cHRlZElkPUEwMzc3MzU4TDJTSUg2SDZKWE9HJmVuY3J5cHRlZEFkSWQ9QTA1OTE1MjJLN1NLQ0o0M1k4Mkkmd2lkZ2V0TmFtZT1zcF9hdGYmYWN0aW9uPWNsaWNrUmVkaXJlY3QmZG9Ob3RMb2dDbGljaz10cnVl&th=1" (id 4) (at 143.51 41.91 0)
+      (effects (font (size 1.27 1.27)) hide)
+    )
+    (pin "1")
+    (pin "2")
+    (pin "3")
   )
   (sheet (at 68.58 35.56) (size 21.59 20.32) (fields_autoplaced)
@@
       (effects (font (size 1.27 1.27)) (justify left bottom))
     )
-    (property "Sheet file" "hierarchical_sheets/fet_output_channel.kicad_sch" (id 1) (at 68.58 56.4646 0)
+    (property "Sheet file" "hierarchical_sheets/fet_output_stage.kicad_sch" (id 1) (at 68.58 56.4646 0)
       (effects (font (size 1.27 1.27)) (justify left top) hide)
     )
@@
   )
   (symbol_instances
-    (path "/23ce54c1-fa71-427d-aa9f-6ac130f31dd0/7f5fcf25-8f29-46fe-8fae-08b9494f1517"
-      (reference "#PWR0101") (unit 1) (value "Earth") (footprint "")
+    (path "/2c9ca97e-d690-4211-b5a5-e2c54d30257c"
+      (reference "#PWR?") (unit 1) (value "Earth") (footprint "")
     )
     (path "/23ce54c1-fa71-427d-aa9f-6ac130f31dd0/8c7b9f57-0d8d-499a-9da5-1e62ee5c82bf"
-      (reference "#PWR0102") (unit 1) (value "GND") (footprint "")
+      (reference "#PWR?") (unit 1) (value "GND") (footprint "")
     )
     (path "/23ce54c1-fa71-427d-aa9f-6ac130f31dd0/272ed9e8-60a6-44e8-871d-08c36f018dec"
-      (reference "D1") (unit 1) (value "LED") (footprint "LED_THT:LED_D5.0mm")
+      (reference "D1") (unit 1) (value "Green") (footprint "LED_THT:LED_D5.0mm")
     )
-    (path "/23ce54c1-fa71-427d-aa9f-6ac130f31dd0/eee2ad48-1403-4d46-af24-ff192c566d6b"
-      (reference "J1") (unit 1) (value "GX16-3") (footprint "")
+    (path "/23ce54c1-fa71-427d-aa9f-6ac130f31dd0/45911c7a-8ef4-45b2-974d-877d27699d8a"
+      (reference "D?") (unit 1) (value "Yellow") (footprint "LED_THT:LED_D5.0mm")
+    )
+    (path "/23ce54c1-fa71-427d-aa9f-6ac130f31dd0/476ffab1-c7f9-4a48-a303-97f0a9f71605"
+      (reference "D?") (unit 1) (value "824500241") (footprint "Diode_SMD:D_SMA")
+    )
+    (path "/23ce54c1-fa71-427d-aa9f-6ac130f31dd0/ed960ca1-422f-4d1c-9c2e-1fda15007d83"
+      (reference "D?") (unit 1) (value "14V") (footprint "Diode_SMD:D_SOD-123")
+    )
+    (path "/e559db9c-9f22-48b9-b3c7-237893391776"
+      (reference "J?") (unit 1) (value "GX16-3") (footprint "")
     )
     (path "/23ce54c1-fa71-427d-aa9f-6ac130f31dd0/2e1c68ea-f0f3-40e7-ae18-ef3fe9534799"
       (reference "Q1") (unit 1) (value "IRF9Z24NPBF") (footprint "DOM:TO-220F-3_Horizontal_TabDown_SMD_PAD")
     )
+    (path "/23ce54c1-fa71-427d-aa9f-6ac130f31dd0/3db9ca56-50ab-49ad-baa1-6e003f5aff4a"
+      (reference "Q?") (unit 1) (value "MMBT3904") (footprint "Package_TO_SOT_SMD:SOT-23")
+    )
+    (path "/23ce54c1-fa71-427d-aa9f-6ac130f31dd0/2075d95a-50bc-4673-8db4-06b1b9bb293e"
+      (reference "R?") (unit 1) (value "1K") (footprint "")
+    )
+    (path "/23ce54c1-fa71-427d-aa9f-6ac130f31dd0/2b401e8b-e0ce-4547-b889-e0b23cf59fe7"
+      (reference "R?") (unit 1) (value "1K") (footprint "")
+    )
+    (path "/23ce54c1-fa71-427d-aa9f-6ac130f31dd0/345e0beb-16e6-4a1b-8c93-27c1aa163d2c"
+      (reference "R?") (unit 1) (value "1K") (footprint "")
+    )
+    (path "/23ce54c1-fa71-427d-aa9f-6ac130f31dd0/69908acb-e426-4ed2-9c22-c705323c8068"
+      (reference "R?") (unit 1) (value "R_US") (footprint "")
+    )
+    (path "/23ce54c1-fa71-427d-aa9f-6ac130f31dd0/af7b0da2-2eb3-4733-8048-0988ef40459c"
+      (reference "R?") (unit 1) (value "R_US") (footprint "")
+    )
+    (path "/23ce54c1-fa71-427d-aa9f-6ac130f31dd0/b4a4e57c-d7bb-49e2-a18c-716d3391b5a2"
+      (reference "R?") (unit 1) (value "1K") (footprint "")
+    )
+    (path "/23ce54c1-fa71-427d-aa9f-6ac130f31dd0/f236bdf5-9e5e-4503-9598-c83c7245169f"
+      (reference "R?") (unit 1) (value "1K") (footprint "")
+    )
+    (path "/23ce54c1-fa71-427d-aa9f-6ac130f31dd0/f4657534-413f-4c4c-abaa-a5f8208ee4d6"
+      (reference "R?") (unit 1) (value "R_US") (footprint "")
+    )
   )

Commit message: Uploading Evil Schemes
Parts:
- removed J?: GX16-3, symbol Connector_Generic:Conn_01x03
Other:
- removed sheet Output Channel
- added sheet DIO 1 (hierarchical_sheets/fet_output_stage.kicad_sch)
- added sheet DIO 10 (hierarchical_sheets/fet_output_stage.kicad_sch)
- added sheet DIO 11 (hierarchical_sheets/fet_output_stage.kicad_sch)
- added sheet DIO 12 (hierarchical_sheets/fet_output_stage.kicad_sch)
- added sheet DIO 2 (hierarchical_sheets/fet_output_stage.kicad_sch)
- added sheet DIO 3 (hierarchical_sheets/fet_output_stage.kicad_sch)
- added sheet DIO 4 (hierarchical_sheets/fet_output_stage.kicad_sch)
- added sheet DIO 5 (hierarchical_sheets/fet_output_stage.kicad_sch)
- added sheet DIO 6 (hierarchical_sheets/fet_output_stage.kicad_sch)
- added sheet DIO 7 (hierarchical_sheets/fet_output_stage.kicad_sch)
- added sheet DIO 8 (hierarchical_sheets/fet_output_stage.kicad_sch)
- added sheet DIO 9 (hierarchical_sheets/fet_output_stage.kicad_sch)
- added sheet GX 16-3 (hierarchical_sheets/digital_output_connector.kicad_sch)
