File: Digital_Output_Module/kicad/digital_output_module.kicad_sch (KiCad schematic)
At the start: 0 parts

Commit message: finished voltage selector switch
Other:
- added sheet Relay Stage (hierarchical_sheets/relay_stage.kicad_sch)
Changed lines of the file:
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@@
   (title_block
     (title "Digital Output Module ")
-    (date "2023-03-27")
+    (date "2023-03-28")
     (rev "1")
     (company "Missouri S&T Rocket Design Team")
     (comment 1 "Seth Sievers")
   )
+  (sheet (at 144.78 64.77) (size 21.59 17.78) (fields_autoplaced)
+    (stroke (width 0.1524) (type solid))
+    (fill (color 255 255 194 1.0000))
+    (property "Sheetname" "Relay Stage" (at 144.78 64.0584 0)
+      (effects (font (size 1.27 1.27)) (justify left bottom))
+    )
+    (property "Sheetfile" "hierarchical_sheets/relay_stage.kicad_sch" (at 144.78 83.1346 0)
+      (effects (font (size 1.27 1.27)) (justify left top))
+    )
+    (instances
+      (project "digital_output_module"
+        (path "/b62c2f25-5357-4427-9763-8fa7314ae7c3" (page "3"))
+      )
+    )
+  )
   (sheet (at 110.49 64.77) (size 20.32 19.05) (fields_autoplaced)
