File: Voltage_Input_Module/Voltage_Input_Module-RevB.kicad_pcb (KiCad board)
At the start: 2 copper layers, 21 parts, among them J1 Conn_01x02, J10 T4140512041-000, J11 Conn_01x02, J12 Conn_01x02, J13 T4140512041-000, J14 T4140512041-000, J15 T4140512041-000, J16 T4140512041-000, J17 T4140512041-000, J18 T4140512041-000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

Commit message: Add files via upload
Parts:
- moved J6 57.8 mm to (45.2, 162.6)
- moved J19 56.1 mm to (42.9, 136.4)
- moved J18 48.3 mm to (42.9, 107.9)
- moved J17 40.9 mm to (42.9, 79.5)
- moved J20 34.5 mm to (42.8, 51.0)
- moved J1 10.5 mm to (108.6, 114.3)
- moved P1 5.08 mm to (143.4, 196.4)
Routing:
- net /4x_4_pin_connector3/power: track 0.00 -> 148.1 mm
- net GND: track 0.00 -> 148.0 mm
- net /AI12-: track 0.00 -> 102.5 mm
- net /AI12+: track 0.00 -> 100.3 mm
- net /AI13-: track 0.00 -> 72.8 mm
- net /AI13+: track 0.00 -> 70.9 mm
- net /AI14-: track 0.00 -> 43.5 mm
- net /AI14+: track 0.00 -> 41.6 mm
- net /AI15-: track 0.00 -> 14.5 mm
- net /AI15+: track 0.00 -> 12.3 mm
