File: Voltage_Input_Module/Voltage_Input_Module-RevB.kicad_sch (KiCad schematic)
At the start: 3 parts, among them J11 Conn_01x02, J12 Conn_01x02, P1 182-037-113R541

Commit message: Add files via upload
Parts:
- added J1, J6: Conn_01x02, powerpole-pp1545:2x_Anderson_Powerpole-25A-S-H-G11, symbol Connector_Generic:Conn_01x02
Connections:
- net GND: now also J1.1 (Pin_1), J6.1 (Pin_1)
- net 4x_4_pin_connector/power_1 renamed 4x_4_pin_connector/power
- net 4x_4_pin_connector1/power_1 renamed 4x_4_pin_connector1/power
- new net 4x_4_pin_connector2/power: J1.2 (Pin_2)
- new net 4x_4_pin_connector3/power: J6.2 (Pin_2)
Other:
- added sheet 4x_4_pin_connector2 (untitled.kicad_sch)
- added sheet 4x_4_pin_connector3 (untitled.kicad_sch)
- sheet 4x_4_pin_connector ports: added power; removed power_1
- sheet 4x_4_pin_connector1 ports: added power; removed power_1
- moved on the sheet: J11, J12, P1
