File: Voltage_Input_Module/untitled.kicad_sch (KiCad schematic)
At the start: 4 parts, among them J10 T4140512041-000, J7 T4140512041-000, J8 T4140512041-000, J9 T4140512041-000

Commit message: Add files via upload
Parts:
- J14: renamed from J8; footprint CONN4_T4140512041 -> Connector_TE-Connectivity:T4140512041-000
- J15: renamed from J9; footprint CONN4_T4140512041 -> Connector_TE-Connectivity:T4140512041-000
- renumbered J7 to J13, J10 to J16
Connections:
- net port_1_signal_in: no longer J13.4, J14.4, J15.4
- net port_1_signal_out: no longer J13.1, J14.1, J15.1
- net power_1 renamed power
- new net port_2_signal_in: J13.4
- new net port_2_signal_out: J13.1
- new net port_3_signal_in: J14.4
- new net port_3_signal_out: J14.1
- new net port_4_signal_in: J15.4
- new net port_4_signal_out: J15.1
Changed lines of the file:
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@@
     (stroke (width 0) (type default) (color 0 0 0 0))
   )
-  (hierarchical_label "port_1_signal_out" (shape output) (at 142.875 108.585 180)
+  (hierarchical_label "port_4_signal_out" (shape output) (at 142.875 108.585 180)
     (effects (font (size 1.27 1.27)) (justify right))
   )
-  (hierarchical_label "port_1_signal_in" (shape input) (at 142.875 100.33 180)
+  (hierarchical_label "port_3_signal_in" (shape input) (at 142.875 100.33 180)
     (effects (font (size 1.27 1.27)) (justify right))
   )
-  (hierarchical_label "port_1_signal_in" (shape input) (at 142.875 122.555 180)
+  (hierarchical_label "port_4_signal_in" (shape input) (at 142.875 122.555 180)
     (effects (font (size 1.27 1.27)) (justify right))
   )
-  (hierarchical_label "port_1_signal_in" (shape input) (at 142.875 77.47 180)
+  (hierarchical_label "port_2_signal_in" (shape input) (at 142.875 77.47 180)
     (effects (font (size 1.27 1.27)) (justify right))
   )
-  (hierarchical_label "power_1" (shape input) (at 140.335 92.075 180)
+  (hierarchical_label "power" (shape input) (at 140.335 92.075 180)
     (effects (font (size 1.27 1.27)) (justify right))
   )
-  (hierarchical_label "power_1" (shape input) (at 140.335 69.215 180)
+  (hierarchical_label "power" (shape input) (at 140.335 69.215 180)
     (effects (font (size 1.27 1.27)) (justify right))
   )
-  (hierarchical_label "port_1_signal_out" (shape output) (at 142.875 86.36 180)
+  (hierarchical_label "port_3_signal_out" (shape output) (at 142.875 86.36 180)
     (effects (font (size 1.27 1.27)) (justify right))
   )
-  (hierarchical_label "power_1" (shape input) (at 140.97 43.815 180)
+  (hierarchical_label "power" (shape input) (at 140.97 43.815 180)
     (effects (font (size 1.27 1.27)) (justify right))
   )
-  (hierarchical_label "power_1" (shape input) (at 140.335 114.3 180)
+  (hierarchical_label "power" (shape input) (at 140.335 114.3 180)
     (effects (font (size 1.27 1.27)) (justify right))
   )
-  (hierarchical_label "port_1_signal_out" (shape output) (at 142.875 63.5 180)
+  (hierarchical_label "port_2_signal_out" (shape output) (at 142.875 63.5 180)
     (effects (font (size 1.27 1.27)) (justify right))
   )
@@
   (symbol (lib_id "TE_Connectivity:T4140512041-000") (at 144.78 89.535 0)
     (in_bom yes) (on_board yes) (fields_autoplaced)
-    (property "Reference" "J8" (id 0) (at 158.75 92.075 0)
+    (property "Reference" "J14" (id 0) (at 158.75 92.075 0)
       (effects (font (size 1.524 1.524)) (justify left))
     )
@@
       (effects (font (size 1.524 1.524)) (justify left))
     )
-    (property "Footprint" "CONN4_T4140512041" (id 2) (at 153.67 79.375 0)
+    (property "Footprint" "Connector_TE-Connectivity:T4140512041-000" (id 2) (at 153.67 79.375 0)
       (effects (font (size 1.524 1.524)) hide)
     )
@@
   (symbol (lib_id "power:GND") (at 140.335 71.755 0)
     (in_bom yes) (on_board yes)
-    (property "Reference" "#PWR0111" (id 0) (at 140.335 78.105 0)
+    (property "Reference" "#PWR0117" (id 0) (at 140.335 78.105 0)
       (effects (font (size 1.27 1.27)) hide)
     )
@@
   (symbol (lib_id "TE_Connectivity:T4140512041-000") (at 144.78 66.675 0)
     (in_bom yes) (on_board yes) (fields_autoplaced)
-    (property "Reference" "J7" (id 0) (at 158.75 69.215 0)
+    (property "Reference" "J13" (id 0) (at 158.75 69.215 0)
       (effects (font (size 1.524 1.524)) (justify left))
     )
@@
   (symbol (lib_id "power:GND") (at 140.335 116.84 0)
     (in_bom yes) (on_board yes)
-    (property "Reference" "#PWR0114" (id 0) (at 140.335 123.19 0)
+    (property "Reference" "#PWR0119" (id 0) (at 140.335 123.19 0)
       (effects (font (size 1.27 1.27)) hide)
     )
@@
   (symbol (lib_id "TE_Connectivity:T4140512041-000") (at 145.415 41.275 0)
     (in_bom yes) (on_board yes) (fields_autoplaced)
-    (property "Reference" "J10" (id 0) (at 159.385 43.815 0)
+    (property "Reference" "J16" (id 0) (at 159.385 43.815 0)
       (effects (font (size 1.524 1.524)) (justify left))
     )
@@
   (symbol (lib_id "TE_Connectivity:T4140512041-000") (at 144.78 111.76 0)
     (in_bom yes) (on_board yes) (fields_autoplaced)
-    (property "Reference" "J9" (id 0) (at 158.75 114.3 0)
+    (property "Reference" "J15" (id 0) (at 158.75 114.3 0)
       (effects (font (size 1.524 1.524)) (justify left))
     )
@@
       (effects (font (size 1.524 1.524)) (justify left))
     )
-    (property "Footprint" "CONN4_T4140512041" (id 2) (at 153.67 101.6 0)
+    (property "Footprint" "Connector_TE-Connectivity:T4140512041-000" (id 2) (at 153.67 101.6 0)
       (effects (font (size 1.524 1.524)) hide)
     )
@@
   (symbol (lib_id "power:GND") (at 140.335 94.615 0)
     (in_bom yes) (on_board yes)
-    (property "Reference" "#PWR0112" (id 0) (at 140.335 100.965 0)
+    (property "Reference" "#PWR0116" (id 0) (at 140.335 100.965 0)
       (effects (font (size 1.27 1.27)) hide)
     )
@@
   (symbol (lib_id "power:GND") (at 140.97 46.355 0)
     (in_bom yes) (on_board yes)
-    (property "Reference" "#PWR0110" (id 0) (at 140.97 52.705 0)
+    (property "Reference" "#PWR0115" (id 0) (at 140.97 52.705 0)
       (effects (font (size 1.27 1.27)) hide)
     )

Commit message: Add files via upload
Parts:
- renumbered J13 to J17, J14 to J18, J15 to J19, J16 to J20
Changed lines of the file:
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@@
   (symbol (lib_id "TE_Connectivity:T4140512041-000") (at 144.78 89.535 0)
     (in_bom yes) (on_board yes) (fields_autoplaced)
-    (property "Reference" "J14" (id 0) (at 158.75 92.075 0)
+    (property "Reference" "J18" (id 0) (at 158.75 92.075 0)
       (effects (font (size 1.524 1.524)) (justify left))
     )
@@
   (symbol (lib_id "power:GND") (at 140.335 71.755 0)
     (in_bom yes) (on_board yes)
-    (property "Reference" "#PWR0117" (id 0) (at 140.335 78.105 0)
+    (property "Reference" "#PWR0122" (id 0) (at 140.335 78.105 0)
       (effects (font (size 1.27 1.27)) hide)
     )
@@
   (symbol (lib_id "TE_Connectivity:T4140512041-000") (at 144.78 66.675 0)
     (in_bom yes) (on_board yes) (fields_autoplaced)
-    (property "Reference" "J13" (id 0) (at 158.75 69.215 0)
+    (property "Reference" "J17" (id 0) (at 158.75 69.215 0)
       (effects (font (size 1.524 1.524)) (justify left))
     )
@@
   (symbol (lib_id "power:GND") (at 140.335 116.84 0)
     (in_bom yes) (on_board yes)
-    (property "Reference" "#PWR0119" (id 0) (at 140.335 123.19 0)
+    (property "Reference" "#PWR0123" (id 0) (at 140.335 123.19 0)
       (effects (font (size 1.27 1.27)) hide)
     )
@@
   (symbol (lib_id "TE_Connectivity:T4140512041-000") (at 145.415 41.275 0)
     (in_bom yes) (on_board yes) (fields_autoplaced)
-    (property "Reference" "J16" (id 0) (at 159.385 43.815 0)
+    (property "Reference" "J20" (id 0) (at 159.385 43.815 0)
       (effects (font (size 1.524 1.524)) (justify left))
     )
@@
   (symbol (lib_id "TE_Connectivity:T4140512041-000") (at 144.78 111.76 0)
     (in_bom yes) (on_board yes) (fields_autoplaced)
-    (property "Reference" "J15" (id 0) (at 158.75 114.3 0)
+    (property "Reference" "J19" (id 0) (at 158.75 114.3 0)
       (effects (font (size 1.524 1.524)) (justify left))
     )
@@
   (symbol (lib_id "power:GND") (at 140.335 94.615 0)
     (in_bom yes) (on_board yes)
-    (property "Reference" "#PWR0116" (id 0) (at 140.335 100.965 0)
+    (property "Reference" "#PWR0121" (id 0) (at 140.335 100.965 0)
       (effects (font (size 1.27 1.27)) hide)
     )
@@
   (symbol (lib_id "power:GND") (at 140.97 46.355 0)
     (in_bom yes) (on_board yes)
-    (property "Reference" "#PWR0115" (id 0) (at 140.97 52.705 0)
+    (property "Reference" "#PWR0124" (id 0) (at 140.97 52.705 0)
       (effects (font (size 1.27 1.27)) hide)
     )
