File: Voltage_Input_Module/kicad/voltage_input_revC/_autosave-voltage_input_revC.kicad_pcb (KiCad board)
At the start: 2 copper layers, 33 parts, among them J1 5747847-4, J10 Conn_01x02, J11 T4143012041-000, J12 Conn_01x02, J13 T4143012041-000, J14 Conn_01x02, J15 T4143012041-000, J16 Conn_01x02, J17 T4143012041-000, J18 Conn_01x02, J19 T4143012041-000, J2 T4143012041-000, J20 Conn_01x02, J21 T4143012041-000, J22 Conn_01x02, J23 T4143012041-000, J24 Conn_01x02, J25 T4143012041-000, J26 Conn_01x02, J27 T4143012041-000, J28 Conn_01x02, J29 T4143012041-000, J3 Conn_01x02, J30 Conn_01x02, J31 T4143012041-000, J32 Conn_01x02, J33 T4143012041-000, J4 Conn_01x02, J5 T4143012041-000, J6 Conn_01x02, J7 T4143012041-000, J8 Conn_01x02, J9 T4143012041-000

Commit message: Started work on trances. Added ground plane, need mounting positions, finish traces, rework/do powerpole connections.
Co-Authored-By: Andrew-Matteson136382 <67286784+Andrew-Matteson136382@users.noreply.github.com>
Routing:
- net /Al12-: track 0.00 -> 181.0 mm
- net /Al12+: track 0.00 -> 177.2 mm
- net /Al13-: track 0.00 -> 142.3 mm
- net /Al13+: track 0.00 -> 138.5 mm
- net /Al14-: track 0.00 -> 103.6 mm
- net /Al14+: track 0.00 -> 99.8 mm
- net /Al15-: track 0.00 -> 64.9 mm
- net /Al15+: track 0.00 -> 61.2 mm
- net /Al11-: track 0.00 -> 2.59 mm
Changed lines of the file:
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@@
       (net 35 "Net-(J3-Pin_2)") (pinfunction "Pin_2") (pintype "passive"))
   )
+  (segment (start 76.043174 141.448174) (end 68.720267 141.448174) (width 0.5) (layer "F.Cu") (net 2))
+  (segment (start 115.4972 176.166542) (end 105.700658 166.37) (width 0.5) (layer "F.Cu") (net 2))
+  (segment (start 105.700658 166.37) (end 100.965 166.37) (width 0.5) (layer "F.Cu") (net 2))
+  (segment (start 100.965 166.37) (end 76.043174 141.448174) (width 0.5) (layer "F.Cu") (net 2))
+  (segment (start 140.701258 163.83) (end 100.965 163.83) (width 0.5) (layer "F.Cu") (net 3))
+  (segment (start 153.0378 176.166542) (end 140.701258 163.83) (width 0.5) (layer "F.Cu") (net 3))
+  (segment (start 75.814574 138.679574) (end 68.720267 138.679574) (width 0.5) (layer "F.Cu") (net 3))
+  (segment (start 100.965 163.83) (end 75.814574 138.679574) (width 0.5) (layer "F.Cu") (net 3))
+  (segment (start 75.585974 135.910974) (end 68.720267 135.910974) (width 0.5) (layer "F.Cu") (net 4))
+  (segment (start 100.965 161.29) (end 75.585974 135.910974) (width 0.5) (layer "F.Cu") (net 4))
+  (segment (start 190.5794 176.166542) (end 175.702858 161.29) (width 0.5) (layer "F.Cu") (net 4))
+  (segment (start 175.702858 161.29) (end 100.965 161.29) (width 0.5) (layer "F.Cu") (net 4))
+  (segment (start 228.12 176.166542) (end 210.703458 158.75) (width 0.5) (layer "F.Cu") (net 5))
+  (segment (start 210.703458 158.75) (end 100.965 158.75) (width 0.5) (layer "F.Cu") (net 5))
+  (segment (start 75.357374 133.142374) (end 68.720267 133.142374) (width 0.5) (layer "F.Cu") (net 5))
+  (segment (start 100.965 158.75) (end 75.357374 133.142374) (width 0.5) (layer "F.Cu") (net 5))
   (segment (start 224.045617 140.860574) (end 225.885368 140.860574) (width 0.5) (layer "F.Cu") (net 9))
   (segment (start 225.885368 140.860574) (end 228.12 138.625942) (width 0.5) (layer "F.Cu") (net 9))
@@
   (segment (start 114.1963 60.197642) (end 115.4972 58.896742) (width 0.5) (layer "F.Cu") (net 18))
   (segment (start 68.720267 94.381974) (end 71.353026 94.381974) (width 0.5) (layer "F.Cu") (net 18))
+  (segment (start 115.4972 179.702074) (end 113.595126 177.8) (width 0.5) (layer "F.Cu") (net 19))
+  (segment (start 111.125 177.8) (end 76.157474 142.832474) (width 0.5) (layer "F.Cu") (net 19))
+  (segment (start 76.157474 142.832474) (end 65.875467 142.832474) (width 0.5) (layer "F.Cu") (net 19))
+  (segment (start 113.595126 177.8) (end 111.125 177.8) (width 0.5) (layer "F.Cu") (net 19))
+  (segment (start 153.0378 179.702074) (end 151.7369 178.401174) (width 0.5) (layer "F.Cu") (net 20))
+  (segment (start 100.965 165.1) (end 75.928874 140.063874) (width 0.5) (layer "F.Cu") (net 20))
+  (segment (start 107.315 165.1) (end 100.965 165.1) (width 0.5) (layer "F.Cu") (net 20))
+  (segment (start 151.731174 178.401174) (end 151.13 177.8) (width 0.5) (layer "F.Cu") (net 20))
+  (segment (start 120.015 177.8) (end 107.315 165.1) (width 0.5) (layer "F.Cu") (net 20))
+  (segment (start 151.13 177.8) (end 120.015 177.8) (width 0.5) (layer "F.Cu") (net 20))
+  (segment (start 75.928874 140.063874) (end 65.875467 140.063874) (width 0.5) (layer "F.Cu") (net 20))
+  (segment (start 151.7369 178.401174) (end 151.731174 178.401174) (width 0.5) (layer "F.Cu") (net 20))
+  (segment (start 75.700274 137.295274) (end 65.875467 137.295274) (width 0.5) (layer "F.Cu") (net 21))
+  (segment (start 190.5794 179.702074) (end 188.677326 177.8) (width 0.5) (layer "F.Cu") (net 21))
+  (segment (start 157.48 177.8) (end 142.24 162.56) (width 0.5) (layer "F.Cu") (net 21))
+  (segment (start 142.24 162.56) (end 100.965 162.56) (width 0.5) (layer "F.Cu") (net 21))
+  (segment (start 100.965 162.56) (end 75.700274 137.295274) (width 0.5) (layer "F.Cu") (net 21))
+  (segment (start 188.677326 177.8) (end 157.48 177.8) (width 0.5) (layer "F.Cu") (net 21))
+  (segment (start 194.945 177.8) (end 177.165 160.02) (width 0.5) (layer "F.Cu") (net 22))
+  (segment (start 177.165 160.02) (end 100.965 160.02) (width 0.5) (layer "F.Cu") (net 22))
+  (segment (start 228.12 179.702074) (end 226.217926 177.8) (width 0.5) (layer "F.Cu") (net 22))
+  (segment (start 226.217926 177.8) (end 194.945 177.8) (width 0.5) (layer "F.Cu") (net 22))
+  (segment (start 75.471674 134.526674) (end 65.875467 134.526674) (width 0.5) (layer "F.Cu") (net 22))
+  (segment (start 100.965 160.02) (end 75.471674 134.526674) (width 0.5) (layer "F.Cu") (net 22))
+  (segment (start 114.1963 140.860574) (end 114.190574 140.860574) (width 0.5) (layer "F.Cu") (net 23))
+  (segment (start 114.190574 140.860574) (end 113.665 140.335) (width 0.5) (layer "F.Cu") (net 23))
+  (segment (start 115.4972 142.161474) (end 114.1963 140.860574) (width 0.5) (layer "F.Cu") (net 23))
   (segment (start 82.55 111.125) (end 78.528526 115.146474) (width 0.5) (layer "F.Cu") (net 27))
   (segment (start 216.967874 111.125) (end 82.55 111.125) (width 0.5) (layer "F.Cu") (net 27))
