File: Voltage_Input_Module/kicad/voltage_input_revC/voltage_input_revC.kicad_pcb (KiCad board)
At the start: 2 copper layers, 33 parts, among them J1 5747847-4, J10 Conn_01x02, J11 T4143012041-000, J12 Conn_01x02, J13 T4143012041-000, J14 Conn_01x02, J15 T4143012041-000, J16 Conn_01x02, J17 T4143012041-000, J18 Conn_01x02, J19 T4143012041-000, J2 T4143012041-000, J20 Conn_01x02, J21 T4143012041-000, J22 Conn_01x02, J23 T4143012041-000, J24 Conn_01x02, J25 T4143012041-000, J26 Conn_01x02, J27 T4143012041-000, J28 Conn_01x02, J29 T4143012041-000, J3 Conn_01x02, J30 Conn_01x02, J31 T4143012041-000, J32 Conn_01x02, J33 T4143012041-000, J4 Conn_01x02, J5 T4143012041-000, J6 Conn_01x02, J7 T4143012041-000, J8 Conn_01x02, J9 T4143012041-000

Commit message: Finished traces, Implemented footprints and 3d models for powerpole connections. Added mounting holes and edge cuts. Need to implement silk screen callouts for sensors.
Co-Authored-By: Andrew-Matteson136382 <67286784+Andrew-Matteson136382@users.noreply.github.com>
Parts:
- J10, J12, J14, J16, J18, J20, J22, J24, J26, J28, J3, J30, J32, J4, J6, J8: footprint custom_libraries:powerpole-1545-2x1 -> MRDT_Connectors:Square_Anderson_2_V_Side_By_Side
- turned J10 to 180 degrees
- turned J12 to 180 degrees
- turned J14 to 180 degrees
- turned J16 to 180 degrees
- turned J18 to 180 degrees
- turned J20 to 180 degrees
- turned J22 to 180 degrees
- turned J24 to 180 degrees
- turned J26 to 180 degrees
- turned J28 to 180 degrees
- turned J3 to 180 degrees
- turned J30 to 180 degrees
- turned J32 to 180 degrees
- turned J4 to 180 degrees
- turned J6 to 180 degrees
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Routing:
- net /Al12-: track 0.00 -> 181.0 mm
- net /Al12+: track 0.00 -> 177.2 mm
- net /Al8-: track 0.00 -> 171.0 mm
- net /Al13-: track 0.00 -> 142.3 mm
- net /Al13+: track 0.00 -> 138.5 mm
- net /Al9-: track 0.00 -> 131.3 mm
- net /Al9+: track 0.00 -> 127.6 mm
- net /Al14-: track 0.00 -> 103.6 mm
- net /Al14+: track 0.00 -> 99.8 mm
- net /Al10-: track 0.00 -> 92.7 mm
- net /Al10+: track 0.00 -> 88.9 mm
- net /Al15-: track 0.00 -> 64.9 mm
- net /Al15+: track 0.00 -> 61.2 mm
- net /Al11-: track 0.00 -> 53.9 mm
- net /Al11+: track 0.00 -> 50.2 mm
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
Commit message: Further reworked traces. Implemented spaces for grounding.
Co-Authored-By: Andrew-Matteson136382 <67286784+Andrew-Matteson136382@users.noreply.github.com>
Parts:
- moved J1 12.7 mm to (70.5, 119.3)
Routing:
- net /Al8+: track 0.00 -> 155.6 mm
- net /Al15-: track 64.9 -> 0.00 mm
- net /Al14-: track 103.6 -> 53.4 mm
- net /Al13-: track 142.3 -> 92.5 mm
- net /Al12-: track 181.0 -> 131.7 mm
- net /Al15+: track 61.2 -> 13.6 mm
- net /Al14+: track 99.8 -> 52.7 mm
- net /Al13+: track 138.5 -> 91.9 mm
- net /Al12+: track 177.2 -> 131.0 mm
- net /Al11-: track 53.9 -> 13.3 mm
- net /Al8-: track 171.0 -> 130.6 mm
- net /Al10-: track 92.7 -> 52.4 mm
- net /Al9-: track 131.3 -> 91.5 mm
- net /Al11+: track 50.2 -> 12.6 mm
- net /Al10+: track 88.9 -> 51.7 mm
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- added copper zone on B.Cu, net GND

Commit message: Finalized traces. Finalized edge cuts. Finalized ground plane. Added vias. Added mounting holes. Added annotations to PCB.
Co-Authored-By: Andrew-Matteson136382 <67286784+Andrew-Matteson136382@users.noreply.github.com>
Parts:
- added REF**: MountingHole_2.2mm_M2, MountingHole:MountingHole_2.2mm_M2, F.Cu at (188.5, 79.4)
- added REF**: Square_Anderson_2_V_Side_By_Side_Symbolic, MRDT_Connectors:Square_Anderson_2_V_Side_By_Side_Symbolic, F.Cu at (88.6, 64.7)
- added REF**: MountingHole_2.2mm_M2, MountingHole:MountingHole_2.2mm_M2, F.Cu at (76.9, 186.1)
- added REF**: MountingHole_2.2mm_M2, MountingHole:MountingHole_2.2mm_M2, F.Cu at (188.4, 159.2)
- added REF**: CONN4_T4143012041_Symbolic, custom_libraries:T4143012041-000_Symbolic, F.Cu at (87.1, 175.9)
- added REF**: MountingHole_2.2mm_M2, MountingHole:MountingHole_2.2mm_M2, F.Cu at (76.8, 49.6)
- added REF**: MountingHole_2.2mm_M2, MountingHole:MountingHole_2.2mm_M2, F.Cu at (292.5, 79.4)
- added REF**: MountingHole_2.2mm_M2, MountingHole:MountingHole_2.2mm_M2, F.Cu at (292.5, 159.2)
- moved J10 14.8 mm to (287.8, 92.6)
- moved J12 14.8 mm to (287.8, 103.4)
- moved J14 14.8 mm to (257.6, 92.6)
- moved J16 14.8 mm to (257.6, 103.4)
- moved J18 14.8 mm to (257.6, 146.0)
- moved J20 14.8 mm to (257.6, 135.2)
- moved J22 14.8 mm to (287.8, 146.0)
- moved J24 14.8 mm to (287.8, 135.2)
- moved J26 14.8 mm to (257.6, 183.5)
- moved J28 14.8 mm to (257.6, 172.7)
- moved J3 14.8 mm to (287.9, 55.1)
- moved J30 14.8 mm to (287.8, 183.5)
- moved J32 14.8 mm to (287.8, 172.7)
- moved J4 14.8 mm to (287.8, 65.9)
- moved J6 14.8 mm to (257.6, 55.1)
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Routing:
- net /Al15-: track 0.00 -> 56.7 mm
- net /Al14-: track 53.4 -> 95.3 mm
- net /Al13-: track 92.5 -> 133.9 mm
- net /Al12-: track 131.7 -> 172.6 mm
- net /Al15+: track 13.6 -> 52.9 mm
- net /Al14+: track 52.7 -> 91.5 mm
- net /Al13+: track 91.9 -> 130.1 mm
- net /Al12+: track 131.0 -> 168.9 mm
- net /Al8-: track 130.6 -> 159.0 mm
- net /Al11-: track 13.3 -> 41.2 mm
- net /Al9-: track 91.5 -> 119.4 mm
- net /Al10-: track 52.4 -> 79.9 mm
- net /Al9+: track 90.8 -> 116.1 mm
- net /Al11+: track 12.6 -> 37.5 mm
- net /Al10+: track 51.7 -> 76.6 mm
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Other:
- board outline added: 234.7 x 149.2 mm
- board text added: "1"
- board text added: "2"
- board text added: "2.2mm"
- board text added: "3"
- board text added: "4"
- board text added: "Al0"
- board text added: "Al0 POWER"
- board text added: "Al1"
- board text added: "Al1 POWER"
- board text added: "Al10"
- board text added: "Al10 POWER"
- board text added: "Al11"
- board text added: "Al11 POWER"
- board text added: "Al12"
- board text added: "Al12 POWER"
- board text added: "Al13"
- board text added: "Al13 POWER"
- board text added: "Al14"
- board text added: "Al14 POWER"
- board text added: "Al15"
- board text added: "Al15 POWER"
- board text added: "Al2"
- board text added: "Al2 POWER"
- board text added: "Al3"
- board text added: "Al3 POWER"
- board text added: "Al4"
- board text added: "Al4 POWER"
- board text added: "Al5"
- board text added: "Al5 POWER"
- board text added: "Al6"
- board text added: "Al6 POWER"
- board text added: "Al7"
- board text added: "Al7 POWER"
- board text added: "Al8"
- board text added: "Al8 POWER"
- board text added: "Al9"
- board text added: "Al9 POWER"
- board text added: "GND(-)"
- board text added: "POWER(+)"
- board text added: "SIGNAL(+)"
- board text added: "SIGNAL(-)"

Commit message: Moved footprints off of vias
Co-Authored-By: Andrew-Matteson136382 <67286784+Andrew-Matteson136382@users.noreply.github.com>
Parts:
- moved REF** 7.17 mm to (86.9, 168.8)
- moved REF** 5.58 mm to (89.0, 59.1)
Changed lines of the file:
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@@
   )
   (footprint "MRDT_Connectors:Square_Anderson_2_V_Side_By_Side_Symbolic" (layer "F.Cu")
-    (at 88.559 64.68 180)
+    (at 88.969 59.12 180)
     (attr through_hole)
     (fp_text reference "REF**" (at 6.2 6.3) (layer "F.SilkS") hide
@@
   )
   (footprint "custom_libraries:T4143012041-000_Symbolic" (layer "F.Cu")
-    (at 87.06 175.94)
+    (at 86.89 168.77)
     (attr through_hole)
     (fp_text reference "REF**" (at 1.6656 8.862133) (layer "F.SilkS") hide
@@
     (effects (font (size 1 1) (thickness 0.15)) (justify left bottom))
   )
-  (gr_text "POWER(+)" (at 72.88 64.44) (layer "F.SilkS")
+  (gr_text "POWER(+)" (at 73.29 58.88) (layer "F.SilkS")
     (effects (font (size 1 1) (thickness 0.15)) (justify left bottom))
   )
@@
     (effects (font (size 1 1) (thickness 0.15)) (justify left bottom))
   )
-  (gr_text "2" (at 84.18 64.48) (layer "F.SilkS")
+  (gr_text "2" (at 84.59 58.92) (layer "F.SilkS")
     (effects (font (size 1 1) (thickness 0.15)) (justify left bottom))
   )
@@
     (effects (font (size 1 1) (thickness 0.15)) (justify left bottom))
   )
-  (gr_text "4" (at 90.24 176.46) (layer "F.SilkS")
+  (gr_text "4" (at 90.07 169.29) (layer "F.SilkS")
     (effects (font (size 1 1) (thickness 0.15)) (justify left bottom))
   )
@@
     (effects (font (size 1 1) (thickness 0.15)) (justify left bottom))
   )
-  (gr_text "1" (at 92.159804 64.286488) (layer "F.SilkS")
+  (gr_text "1" (at 92.569804 58.726488) (layer "F.SilkS")
     (effects (font (size 1 1) (thickness 0.15)) (justify left bottom))
   )
@@
     (effects (font (size 1 1) (thickness 0.15)) (justify left bottom))
   )
-  (gr_text "POWER(+)" (at 76.03 180.92) (layer "F.SilkS")
+  (gr_text "POWER(+)" (at 75.86 173.75) (layer "F.SilkS")
     (effects (font (size 1 1) (thickness 0.15)) (justify left bottom))
   )
@@
     (effects (font (size 1 1) (thickness 0.15)) (justify left bottom))
   )
-  (gr_text "GND(-)" (at 77.37 176.6) (layer "F.SilkS")
+  (gr_text "GND(-)" (at 77.2 169.43) (layer "F.SilkS")
     (effects (font (size 1 1) (thickness 0.15)) (justify left bottom))
   )
@@
     (effects (font (size 1 1) (thickness 0.15)) (justify left bottom))
   )
-  (gr_text "SIGNAL(+)" (at 94.46 175.74) (layer "F.SilkS")
+  (gr_text "SIGNAL(+)" (at 94.29 168.57) (layer "F.SilkS")
     (effects (font (size 1 1) (thickness 0.15)) (justify left bottom))
   )
-  (gr_text "2" (at 86.59 180.18) (layer "F.SilkS")
+  (gr_text "2" (at 86.42 173.01) (layer "F.SilkS")
     (effects (font (size 1 1) (thickness 0.15)) (justify left bottom))
   )
@@
     (effects (font (size 1 1) (thickness 0.15)) (justify left bottom))
   )
-  (gr_text "3" (at 86.54 176.51) (layer "F.SilkS")
+  (gr_text "3" (at 86.37 169.34) (layer "F.SilkS")
     (effects (font (size 1 1) (thickness 0.15)) (justify left bottom))
   )
-  (gr_text "SIGNAL(-)" (at 94.46 179.94) (layer "F.SilkS")
+  (gr_text "SIGNAL(-)" (at 94.29 172.77) (layer "F.SilkS")
     (effects (font (size 1 1) (thickness 0.15)) (justify left bottom))
   )
@@
     (effects (font (size 1 1) (thickness 0.15)) (justify left bottom))
   )
-  (gr_text "GND(-)" (at 97.67 64.55) (layer "F.SilkS")
+  (gr_text "GND(-)" (at 98.08 58.99) (layer "F.SilkS")
     (effects (font (size 1 1) (thickness 0.15)) (justify left bottom))
   )
