File: AI_Board_RevA/AI_Board_RevA.kicad_pcb (KiCad board)
At the start: 2 copper layers, 33 parts, among them J0 Conn_01x04, J1 Conn_01x04, J10 Conn_01x04, J11 Conn_01x04, J12 Conn_01x04, J13 Conn_01x04, J14 Conn_01x04, J15 Conn_01x04, J16 DB37_Female, J17 Conn_01x02, J18 Conn_01x02, J19 Conn_01x02, J2 Conn_01x04, J20 Conn_01x02, J21 Conn_01x02, J22 Conn_01x02, J23 Conn_01x02, J24 Conn_01x02, J25 Conn_01x02, J26 Conn_01x02, J27 Conn_01x02, J28 Conn_01x02, J29 Conn_01x02, J3 Conn_01x04, J30 Conn_01x02, J31 Conn_01x02, J32 Conn_01x02, J4 Conn_01x04, J5 Conn_01x04, J6 Conn_01x04, J7 Conn_01x04, J8 Conn_01x04, J9 Conn_01x04

Commit message: Penultimate draft
Parts:
- added REF**: MountingHole_3.2mm_M3_DIN965, MountingHole:MountingHole_3.2mm_M3_DIN965, F.Cu at (48.0, 32.0)
- added REF**: MountingHole_3.2mm_M3_DIN965, MountingHole:MountingHole_3.2mm_M3_DIN965, F.Cu at (254.0, 227.0)
- added REF**: MountingHole_3.2mm_M3_DIN965, MountingHole:MountingHole_3.2mm_M3_DIN965, F.Cu at (48.0, 227.0)
- added REF**: MountingHole_3.2mm_M3_DIN965, MountingHole:MountingHole_3.2mm_M3_DIN965, F.Cu at (48.0, 129.5)
- added REF**: MountingHole_3.2mm_M3_DIN965, MountingHole:MountingHole_3.2mm_M3_DIN965, F.Cu at (254.0, 32.0)
- added REF**: MountingHole_3.2mm_M3_DIN965, MountingHole:MountingHole_3.2mm_M3_DIN965, F.Cu at (254.0, 129.5)
- moved J12 92.0 mm to (122.5, 191.7), turned to 180 degrees
- moved J8 90.4 mm to (123.8, 144.3), turned to 180 degrees
- moved J13 88.6 mm to (155.5, 192.3), turned to -90 degrees
- moved J17 87.9 mm to (125.0, 64.4), turned to 180 degrees
- moved J9 86.9 mm to (157.7, 144.4), turned to -90 degrees
- moved J14 85.0 mm to (190.3, 192.4), turned to -90 degrees
- moved J22 84.5 mm to (159.2, 105.1), turned to 180 degrees
- moved J25 84.3 mm to (122.4, 126.5)
- moved J18 84.2 mm to (159.6, 63.2), turned to 180 degrees
- moved J29 84.0 mm to (121.5, 173.4)
- moved J21 83.8 mm to (120.7, 104.2)
- moved J10 83.4 mm to (194.2, 144.8), turned to -90 degrees
- moved J4 83.2 mm to (123.1, 90.0), turned to 180 degrees
- moved J0 82.8 mm to (123.3, 46.1), turned to 180 degrees
- moved J15 81.5 mm to (224.1, 192.6), turned to -90 degrees
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Connections:
- J0 pad 3: /COM -> GND
- J0 pad 4: +24V -> Net-(J0-Pin_4)
- J1 pad 3: /COM -> GND
- J1 pad 4: +24V -> Net-(J1-Pin_4)
- J10 pad 3: /COM -> GND
- J10 pad 4: +24V -> Net-(J10-Pin_4)
- J11 pad 3: /COM -> GND
- J11 pad 4: +24V -> Net-(J11-Pin_4)
- J12 pad 3: /COM -> GND
- J12 pad 4: +24V -> Net-(J12-Pin_4)
- J13 pad 3: /COM -> GND
- J13 pad 4: +24V -> Net-(J13-Pin_4)
- J14 pad 3: /COM -> GND
- J14 pad 4: +24V -> Net-(J14-Pin_4)
- J15 pad 3: /COM -> GND
- J15 pad 4: +24V -> Net-(J15-Pin_4)
- J17 pad 1: +24V -> GND
- J17 pad 2: GND -> Net-(J0-Pin_4)
- J18 pad 1: +24V -> GND
- J18 pad 2: GND -> Net-(J1-Pin_4)
- J19 pad 1: +24V -> GND
- J19 pad 2: GND -> Net-(J19-Pin_2)
- J2 pad 3: /COM -> GND
- J2 pad 4: +24V -> Net-(J19-Pin_2)
- J20 pad 1: +24V -> GND
- J20 pad 2: GND -> Net-(J20-Pin_2)
- J21 pad 1: +24V -> GND
- J21 pad 2: GND -> Net-(J21-Pin_2)
- J22 pad 1: +24V -> GND
- J22 pad 2: GND -> Net-(J22-Pin_2)
- J23 pad 1: +24V -> GND
- J23 pad 2: GND -> Net-(J23-Pin_2)
- J24 pad 1: +24V -> GND
- J24 pad 2: GND -> Net-(J24-Pin_2)
- J25 pad 1: +24V -> GND
- J25 pad 2: GND -> Net-(J25-Pin_2)
- J26 pad 1: +24V -> GND
- J26 pad 2: GND -> Net-(J26-Pin_2)
- J27 pad 1: +24V -> GND
- J27 pad 2: GND -> Net-(J10-Pin_4)
- J28 pad 1: +24V -> GND
- J28 pad 2: GND -> Net-(J11-Pin_4)
- J29 pad 1: +24V -> GND
- J29 pad 2: GND -> Net-(J12-Pin_4)
- J3 pad 3: /COM -> GND
- J3 pad 4: +24V -> Net-(J20-Pin_2)
- J30 pad 1: +24V -> GND
- J30 pad 2: GND -> Net-(J13-Pin_4)
- J31 pad 1: +24V -> GND
- J31 pad 2: GND -> Net-(J14-Pin_4)
- J32 pad 1: +24V -> GND
- J32 pad 2: GND -> Net-(J15-Pin_4)
- J4 pad 3: /COM -> GND
- J4 pad 4: +24V -> Net-(J21-Pin_2)
- J5 pad 3: /COM -> GND
- J5 pad 4: +24V -> Net-(J22-Pin_2)
- J6 pad 3: /COM -> GND
- J6 pad 4: +24V -> Net-(J23-Pin_2)
- J7 pad 3: /COM -> GND
- J7 pad 4: +24V -> Net-(J24-Pin_2)
- J8 pad 3: /COM -> GND
- J8 pad 4: +24V -> Net-(J25-Pin_2)
- J9 pad 3: /COM -> GND
- J9 pad 4: +24V -> Net-(J26-Pin_2)
Routing:
- net /AI15-: track 0.00 -> 230.1 mm
- net /AI15+: track 0.00 -> 215.9 mm
- net /AI11-: track 0.00 -> 195.0 mm
- net /AI14-: track 0.00 -> 188.3 mm
- net /AI3-: track 0.00 -> 188.2 mm
- net /AI3+: track 0.00 -> 186.4 mm
- net /AI11+: track 0.00 -> 185.0 mm
- net /AI7-: track 0.00 -> 175.9 mm
- net /AI14+: track 0.00 -> 175.2 mm
- net /AI7+: track 0.00 -> 171.1 mm
- net /AI2-: track 0.00 -> 156.7 mm
- net /AI10-: track 0.00 -> 156.1 mm
- net /AI2+: track 0.00 -> 154.6 mm
- net /AI10+: track 0.00 -> 146.2 mm
- net /AI13-: track 0.00 -> 144.7 mm
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- added copper zone on B.Cu, net GND
- added copper zone on F.Cu, net GND
Other:
- board outline added: 222 x 211 mm
- board text added: "AI0+"
- board text added: "AI0-"
- board text added: "ExcIn"
- board text added: "GND"
- board text added: "Missouri S&T RDT"
- board text added: "Rakshak Sudhakaran"
