File: AI_Board_RevA/AI_Board_RevA.kicad_sch (KiCad schematic)
At the start: 33 parts, among them J0 Conn_01x04, J1 Conn_01x04, J10 Conn_01x04, J11 Conn_01x04, J12 Conn_01x04, J13 Conn_01x04, J14 Conn_01x04, J15 Conn_01x04, J16 DB37_Female, J17 Conn_01x02, J18 Conn_01x02, J19 Conn_01x02, J2 Conn_01x04, J20 Conn_01x02, J21 Conn_01x02, J22 Conn_01x02, J23 Conn_01x02, J24 Conn_01x02, J25 Conn_01x02, J26 Conn_01x02, J27 Conn_01x02, J28 Conn_01x02, J29 Conn_01x02, J3 Conn_01x04, J30 Conn_01x02, J31 Conn_01x02, J32 Conn_01x02, J4 Conn_01x04, J5 Conn_01x04, J6 Conn_01x04, J7 Conn_01x04, J8 Conn_01x04, J9 Conn_01x04

Commit message: Penultimate draft
Parts:
- J16: footprint Connector_Dsub:DSUB-37_Female_EdgeMount_P2.77mm -> Connector_Dsub:DSUB-37_Female_Vertical_P2.77x2.84mm_MountingHoles
Connections:
- net COM: no longer J0.3 (Pin_3), J1.3 (Pin_3), J10.3 (Pin_3), J11.3 (Pin_3), J12.3 (Pin_3), J13.3 (Pin_3), J14.3 (Pin_3), J15.3 (Pin_3), J2.3 (Pin_3), J3.3 (Pin_3), J4.3 (Pin_3), J5.3 (Pin_3), J6.3 (Pin_3), J7.3 (Pin_3), J8.3 (Pin_3), J9.3 (Pin_3)
- net GND: now also J0.3 (Pin_3), J1.3 (Pin_3), J10.3 (Pin_3), J11.3 (Pin_3), J12.3 (Pin_3), J13.3 (Pin_3), J14.3 (Pin_3), J15.3 (Pin_3), J17.1 (Pin_1), J18.1 (Pin_1), J19.1 (Pin_1), J2.3 (Pin_3), J20.1 (Pin_1), J21.1 (Pin_1), J22.1 (Pin_1), J23.1 (Pin_1), J24.1 (Pin_1), J25.1 (Pin_1), J26.1 (Pin_1), J27.1 (Pin_1), J28.1 (Pin_1), J29.1 (Pin_1), J3.3 (Pin_3), J30.1 (Pin_1), J31.1 (Pin_1), J32.1 (Pin_1), J4.3 (Pin_3), J5.3 (Pin_3), J6.3 (Pin_3), J7.3 (Pin_3), J8.3 (Pin_3), J9.3 (Pin_3); no longer J17.2 (Pin_2), J18.2 (Pin_2), J19.2 (Pin_2), J20.2 (Pin_2), J21.2 (Pin_2), J22.2 (Pin_2), J23.2 (Pin_2), J24.2 (Pin_2), J25.2 (Pin_2), J26.2 (Pin_2), J27.2 (Pin_2), J28.2 (Pin_2), J29.2 (Pin_2), J30.2 (Pin_2), J31.2 (Pin_2), J32.2 (Pin_2)
- removed net +24V: J0.4 (Pin_4), J1.4 (Pin_4), J10.4 (Pin_4), J11.4 (Pin_4), J12.4 (Pin_4), J13.4 (Pin_4), J14.4 (Pin_4), J15.4 (Pin_4), J17.1 (Pin_1), J18.1 (Pin_1), J19.1 (Pin_1), J2.4 (Pin_4), J20.1 (Pin_1), J21.1 (Pin_1), J22.1 (Pin_1), J23.1 (Pin_1), J24.1 (Pin_1), J25.1 (Pin_1), J26.1 (Pin_1), J27.1 (Pin_1), J28.1 (Pin_1), J29.1 (Pin_1), J3.4 (Pin_4), J30.1 (Pin_1), J31.1 (Pin_1), J32.1 (Pin_1), J4.4 (Pin_4), J5.4 (Pin_4), J6.4 (Pin_4), J7.4 (Pin_4), J8.4 (Pin_4), J9.4 (Pin_4)
- new net: J14.4 (Pin_4), J31.2 (Pin_2)
- new net: J13.4 (Pin_4), J30.2 (Pin_2)
- new net: J24.2 (Pin_2), J7.4 (Pin_4)
- new net: J11.4 (Pin_4), J28.2 (Pin_2)
- new net: J23.2 (Pin_2), J6.4 (Pin_4)
- new net: J19.2 (Pin_2), J2.4 (Pin_4)
- new net: J26.2 (Pin_2), J9.4 (Pin_4)
- new net: J1.4 (Pin_4), J18.2 (Pin_2)
- new net: J22.2 (Pin_2), J5.4 (Pin_4)
- new net: J0.4 (Pin_4), J17.2 (Pin_2)
- new net: J21.2 (Pin_2), J4.4 (Pin_4)
- new net: J20.2 (Pin_2), J3.4 (Pin_4)
- new net: J10.4 (Pin_4), J27.2 (Pin_2)
- new net: J25.2 (Pin_2), J8.4 (Pin_4)
- new net: J12.4 (Pin_4), J29.2 (Pin_2)
- new net: J15.4 (Pin_4), J32.2 (Pin_2)
- no-connect marks 0 -> 5
